File: PCBs/LV_PCB/LV_PCB.kicad_sch (KiCad schematic)
At the start: 144 parts

Commit message: update schematics snapshot
Parts:
- removed 10uF?: 10uF, Capacitor_THT:CP_Radial_D8.0mm_P3.50mm, symbol Device:C_Polarized
- removed AE?: GPS, footprint:ANTENA, symbol Device:Antenna
- removed C? (x4): 1nF, Capacitor_THT:C_Disc_D3.0mm_W2.0mm_P2.50mm, symbol Device:C_Small
- removed C? (x2): 100uF, Capacitor_THT:CP_Radial_D8.0mm_P3.50mm, symbol Device:C_Polarized_Small
- removed D?: OK_{LV, LED_THT:LED_D5.0mm, symbol Device:LED
- removed D?: OK_{AUX, LED_THT:LED_D5.0mm, symbol Device:LED
- removed D?: OK_{IMD, LED_THT:LED_D5.0mm, symbol Device:LED
- removed D?: FAULT_{BSPD, LED_THT:LED_D5.0mm, symbol Device:LED
- removed D?: FAULT_{BMS, LED_THT:LED_D5.0mm, symbol Device:LED
- removed D?: LED5, LED_THT:LED_D5.0mm, symbol Device:LED
- removed D?: LED3, LED_THT:LED_D5.0mm, symbol Device:LED
- removed D?: OK_{HV, LED_THT:LED_D5.0mm, symbol Device:LED
- removed D?: OK_{BSPD, LED_THT:LED_D5.0mm, symbol Device:LED
- removed D?: RTD, LED_THT:LED_D5.0mm, symbol Device:LED
- removed D?: LED0, LED_THT:LED_D5.0mm, symbol Device:LED
- removed D?: BSPD_GATE, LED_THT:LED_D5.0mm, symbol Device:LED
- removed D?: LED1, LED_THT:LED_D5.0mm, symbol Device:LED
- removed D?: FAULT_{IMD, LED_THT:LED_D5.0mm, symbol Device:LED
- removed D?: LED4, LED_THT:LED_D5.0mm, symbol Device:LED
- removed D?: OK_{BMS, LED_THT:LED_D5.0mm, symbol Device:LED
- removed D?: LED2, LED_THT:LED_D5.0mm, symbol Device:LED
- removed F?: 8A, footprint:Fuse_Holder(GF-205B), symbol Device:Fuse
- removed J? (x2): 5267-16AX, symbol Connector:Conn_01x16_Female
- removed J?: 5267-08AX, symbol Connector:Conn_01x08_Female
- removed J?: 5267-06AX, symbol Connector:Conn_01x06_Female
- removed J?: Conn_01x06_Male, symbol Connector:Conn_01x06_Male
- removed J? (x2): 5267-12AX, symbol Connector:Conn_01x12_Female
- removed J?: HIGH_CURRENT, symbol Connector:Conn_01x08_Female
- removed J?: Conn_01x02_Female, symbol 11:Conn_01x02_Female
- removed J? (x2): 5267-10AX, symbol Connector:Conn_01x10_Female
- removed K? (x5): HR702NH-DC12V, footprint:HR702, symbol Relay:DIPxx-1Cxx-51x
- removed K?: HR90L2_12V, footprint:HR90L2, symbol Relay:EC2-3TNU
- removed Q? (x3): 2N3904, Package_TO_SOT_THT:TO-92_Inline_Wide, symbol Device:Q_NPN_CBE
- removed Q?: IRF640, footprint:IRF640NPBF, symbol Device:Q_NMOS_GDS
- removed Q? (x7): 2N3904, Package_TO_SOT_THT:TO-92_Inline_Wide, symbol Transistor_BJT:2N3904
- removed Q?: IRF9540N, Package_TO_SOT_THT:TO-220-3_Vertical, symbol Transistor_FET:IRF9540N
- removed Q? (x2): IRF640, footprint:IRF640NPBF, symbol Transistor_FET:IRF740
- removed R? (x2): 4M, Resistor_THT:R_Axial_DIN0207_L6.3mm_D2.5mm_P10.16mm_Horizontal, symbol Device:R_US
- removed R? (x18): 10k, Resistor_THT:R_Axial_DIN0207_L6.3mm_D2.5mm_P10.16mm_Horizontal, symbol Device:R_US
- removed R? (x17): 1k, Resistor_THT:R_Axial_DIN0207_L6.3mm_D2.5mm_P10.16mm_Horizontal, symbol Device:R_US
- removed R? (x10): 100, Resistor_THT:R_Axial_DIN0207_L6.3mm_D2.5mm_P10.16mm_Horizontal, symbol Device:R_US
- removed R? (x6): 2.7k, Resistor_THT:R_Axial_DIN0207_L6.3mm_D2.5mm_P10.16mm_Horizontal, symbol Device:R_US
- removed R?: 240K, Resistor_THT:R_Axial_DIN0207_L6.3mm_D2.5mm_P10.16mm_Horizontal, symbol Device:R_US
- removed R?: 3.3k, Resistor_THT:R_Axial_DIN0207_L6.3mm_D2.5mm_P10.16mm_Horizontal, symbol Device:R_US
- removed R?: 51k, Resistor_THT:R_Axial_DIN0207_L6.3mm_D2.5mm_P10.16mm_Horizontal, symbol Device:R_US
- removed R?: 4.7k, Resistor_THT:R_Axial_DIN0207_L6.3mm_D2.5mm_P10.16mm_Horizontal, symbol Device:R_US
- removed R?: 200k, Resistor_THT:R_Axial_DIN0207_L6.3mm_D2.5mm_P10.16mm_Horizontal, symbol Device:R_US
- removed RLY?: RLY_{BSPD, footprint:RT424F12, symbol A-FA_PARTS:RT424F12
- removed RLY?: RLY_{BMS, footprint:RT424F12, symbol A-FA_PARTS:RT424F12
- removed RLY?: RLY_{IMD, footprint:RT424F12, symbol A-FA_PARTS:RT424F12
- removed RV?: TUNE_{HALL, Potentiometer_THT:Potentiometer_Bourns_3296W_Vertical, symbol Device:R_Potentiometer_US
- removed RV?: TUNE_{BRAKE, Potentiometer_THT:Potentiometer_Bourns_3296W_Vertical, symbol Device:R_Potentiometer_US
- removed SW?: CAN_{DEBUG, footprint:TOGGLE_SWITCH, symbol Switch:SW_DPST
- removed SW?: CAN_{ECU, footprint:TOGGLE_SWITCH, symbol Switch:SW_DPST
- removed SW?: CAN_{LOGGER, footprint:TOGGLE_SWITCH, symbol Switch:SW_DPST
- removed SW?: CAN_{BMS, footprint:TOGGLE_SWITCH, symbol Switch:SW_DPST
- removed SW?: ESP_{PROGRAM, footprint:TACT_SWITCH, symbol Switch:SW_Push
- removed SW?: CAN_{INV, footprint:TOGGLE_SWITCH, symbol Switch:SW_DPST
- removed SW?: PROGRAM, footprint:TACT_SWITCH, symbol Switch:SW_Push
- removed SW?: ESP_{RST, footprint:TACT_SWITCH, symbol Switch:SW_Push
- removed SW?: \PROG_ENA, footprint:TACT_SWITCH, symbol Switch:SW_Push
- removed U?: ESP32-WROOM-32D, footprint:MODULE_ESP32-WROOM-32D, symbol ESP32-WROOM-32D:ESP32-WROOM-32D
- removed U? (x2): LM555xN, footprint:NE555P, symbol Timer:LM555xN
- removed U?: 5V Converter, footprint:DCDC_MODULE, symbol A-FA_PARTS:DC-DC_Converter
- removed U?: STM32F407VETx, footprint:STM32F407_HOLDER, symbol MCU_ST_STM32F4:STM32F407VETx
- removed U?: AMS1117-5.0, footprint:AMS1117-5.0, symbol Regulator_Linear:AMS1117-5.0
- removed U?: DFR0299, footprint:DFR0299, symbol DFR0299:DFR0299
- removed U?: CAN_TRANSCEIVER, footprint:CAN_TRANSIVER, symbol A-FA_PARTS:CAN_TRANSCEIVER
- removed U? (x2): LM311, footprint:LM311P, symbol Comparator:LM311
- removed U?: ADXL345, footprint:ADXL345, symbol A-FA_PARTS:ADXL345
- removed U?: NE555D, footprint:NE555P, symbol Timer:NE555D
- removed U?: D302, footprint:SPK_D302, symbol A-FA_PARTS:D302
- removed U?: NEO-7M, footprint:GPSV3-NE0, symbol A-FA_PARTS:NEO-7M
- removed U?: 3.3V Converter, footprint:DCDC_MODULE, symbol A-FA_PARTS:DC-DC_Converter
- added 10uF1: 10uF, Capacitor_THT:CP_Radial_D5.0mm_P2.50mm, symbol Device:C_Polarized
- added AE1: GPS, footprint:ANTENA, symbol Device:Antenna
- added C1, C2, C3, C4: 1nF, Capacitor_THT:C_Disc_D5.0mm_W2.5mm_P2.50mm, symbol Device:C_Small
- added C5, C6: 100uF, Capacitor_THT:CP_Radial_D5.0mm_P2.50mm, symbol Device:C_Polarized_Small
- added D1: OK_{LV, LED_THT:LED_D5.0mm, symbol Device:LED
- added D10: OK_{HV, LED_THT:LED_D5.0mm, symbol Device:LED
- added D11: LED0, LED_THT:LED_D5.0mm, symbol Device:LED
- added D12: LED1, LED_THT:LED_D5.0mm, symbol Device:LED
- added D13: LED2, LED_THT:LED_D5.0mm, symbol Device:LED
- added D14: LED3, LED_THT:LED_D5.0mm, symbol Device:LED
- added D15: LED4, LED_THT:LED_D5.0mm, symbol Device:LED
- added D16: LED5, LED_THT:LED_D5.0mm, symbol Device:LED
- added D17: RTD, LED_THT:LED_D5.0mm, symbol Device:LED
- added D2: FAULT_{BMS, LED_THT:LED_D5.0mm, symbol Device:LED
- added D3: OK_{AUX, LED_THT:LED_D5.0mm, symbol Device:LED
- added D4: OK_{BMS, LED_THT:LED_D5.0mm, symbol Device:LED
- added D5: FAULT_{IMD, LED_THT:LED_D5.0mm, symbol Device:LED
- added D6: OK_{IMD, LED_THT:LED_D5.0mm, symbol Device:LED
- added D7: FAULT_{BSPD, LED_THT:LED_D5.0mm, symbol Device:LED
- added D8: OK_{BSPD, LED_THT:LED_D5.0mm, symbol Device:LED
- added D9: BSPD_GATE, LED_THT:LED_D5.0mm, symbol Device:LED
- added F1: 8A, Fuse:Fuseholder_Cylinder-5x20mm_Stelvio-Kontek_PTF78_Horizontal_Open, symbol Device:Fuse
- added J1, J2: 5267-12AX, Connector_PinHeader_2.54mm:PinHeader_1x12_P2.54mm_Vertical, symbol Connector:Conn_01x12_Female
- added J10, J9: 5267-10AX, Connector_PinHeader_2.54mm:PinHeader_1x10_P2.54mm_Vertical, symbol Connector:Conn_01x10_Female
- added J11: Conn_01x06_Male, Connector_PinHeader_2.54mm:PinHeader_1x06_P2.54mm_Vertical, symbol Connector:Conn_01x06_Male
- added J12: Conn_01x01_Male, Connector_PinSocket_2.54mm:PinSocket_1x01_P2.54mm_Vertical, symbol 11:Conn_01x01_Male
- added J3: 5267-08AX, footprint:5566-08, symbol Connector:Conn_01x08_Female
- added J4: HIGH_CURRENT, footprint:5566-08, symbol Connector:Conn_01x08_Female
- added J5, J8: 5267-16AX, Connector_PinHeader_2.54mm:PinHeader_1x16_P2.54mm_Vertical, symbol Connector:Conn_01x16_Female
- added J6: Conn_01x02_Female, footprint:5566-02A, symbol 11:Conn_01x02_Female
- added J7: 5267-06AX, Connector_PinHeader_2.54mm:PinHeader_1x06_P2.54mm_Vertical, symbol Connector:Conn_01x06_Female
- added K1, K2, K3, K4, K5: HR702NH-DC12V, footprint:HR702, symbol Relay:DIPxx-1Cxx-51x
- added K6: HR90L2_12V, footprint:HR90L2, symbol Relay:EC2-3TNU
- added Q1: IRF640, footprint:IRF640NPBF, symbol Device:Q_NMOS_GDS
- added Q10, Q14, Q5, Q6, Q7, Q8, Q9: 2N3904, Package_TO_SOT_THT:TO-92_Inline_Wide, symbol Transistor_BJT:2N3904
- added Q11, Q12, Q13: 2N3904, Package_TO_SOT_THT:TO-92_Inline_Wide, symbol Device:Q_NPN_CBE
- added Q2, Q4: IRF640, footprint:IRF640NPBF, symbol Transistor_FET:IRF740
- added Q3: IRF9540N, Package_TO_SOT_THT:TO-220-3_Vertical, symbol Transistor_FET:IRF9540N
- added R1, R10, R11, R13, R14, R15, R16, R19, R25, R33, R34, R35, R36, R4, R48, R49, R55: 1k, Resistor_THT:R_Axial_DIN0207_L6.3mm_D2.5mm_P10.16mm_Horizontal, symbol Device:R_US
- added R12, R2, R20, R21, R24, R26, R27, R28, R29, R3, R30, R31, R32, R37, R44, R45, R47, R51: 10k, Resistor_THT:R_Axial_DIN0207_L6.3mm_D2.5mm_P10.16mm_Horizontal, symbol Device:R_US
- added R17: 200k, Resistor_THT:R_Axial_DIN0207_L6.3mm_D2.5mm_P10.16mm_Horizontal, symbol Device:R_US
- added R18: 51k, Resistor_THT:R_Axial_DIN0207_L6.3mm_D2.5mm_P10.16mm_Horizontal, symbol Device:R_US
- added R22, R23: 4M, Resistor_THT:R_Axial_DIN0207_L6.3mm_D2.5mm_P10.16mm_Horizontal, symbol Device:R_US
- added R38, R39, R40, R41, R42, R43, R5, R6, R7, R8: 100, Resistor_THT:R_Axial_DIN0207_L6.3mm_D2.5mm_P10.16mm_Horizontal, symbol Device:R_US
- added R46: 3.3k, Resistor_THT:R_Axial_DIN0207_L6.3mm_D2.5mm_P10.16mm_Horizontal, symbol Device:R_US
- added R50: 4.7k, Resistor_THT:R_Axial_DIN0207_L6.3mm_D2.5mm_P10.16mm_Horizontal, symbol Device:R_US
- added R52, R53, R54, R56, R57, R58: 2.7k, Resistor_THT:R_Axial_DIN0207_L6.3mm_D2.5mm_P10.16mm_Horizontal, symbol Device:R_US
- added R9: 240K, Resistor_THT:R_Axial_DIN0207_L6.3mm_D2.5mm_P10.16mm_Horizontal, symbol Device:R_US
- added RLY1: RLY_{BMS, footprint:RT424F12, symbol A-FA_PARTS:RT424F12
- added RLY2: RLY_{IMD, footprint:RT424F12, symbol A-FA_PARTS:RT424F12
- added RLY3: RLY_{BSPD, footprint:RT424F12, symbol A-FA_PARTS:RT424F12
- added RV1: TUNE_{BRAKE, Potentiometer_THT:Potentiometer_Bourns_3296W_Vertical, symbol Device:R_Potentiometer_US
- added RV2: TUNE_{HALL, Potentiometer_THT:Potentiometer_Bourns_3296W_Vertical, symbol Device:R_Potentiometer_US
- added SW2: ESP_{RST, footprint:TACT_SWITCH, symbol Switch:SW_Push
- added SW3: CAN_{BMS, footprint:TOGGLE_SWITCH, symbol Switch:SW_DPST
- added SW4: CAN_{INV, footprint:TOGGLE_SWITCH, symbol Switch:SW_DPST
- added SW5: CAN_{LOGGER, footprint:TOGGLE_SWITCH, symbol Switch:SW_DPST
- added SW6: CAN_{ECU, footprint:TOGGLE_SWITCH, symbol Switch:SW_DPST
- added SW7: CAN_{DEBUG, footprint:TOGGLE_SWITCH, symbol Switch:SW_DPST
- added SW8: ESP_{PROGRAM, footprint:TACT_SWITCH, symbol Switch:SW_Push
- added SW9: PROGRAM, footprint:TACT_SWITCH, symbol Switch:SW_Push
- added U1: NE555D, footprint:NE555P, symbol Timer:NE555D
- added U10: NEO-7M, footprint:GPSV3-NE0, symbol A-FA_PARTS:NEO-7M
- added U11: ESP32-WROOM-32D, footprint:MODULE_ESP32-WROOM-32D, symbol ESP32-WROOM-32D:ESP32-WROOM-32D
- added U12: DFR0299, footprint:DFR0299, symbol DFR0299:DFR0299
- added U13, U14: LM555xN, footprint:NE555P, symbol Timer:LM555xN
- added U15: STM32F407VETx, footprint:STM32F407_HOLDER, symbol MCU_ST_STM32F4:STM32F407VETx
- added U2, U3: LM311, footprint:LM311P, symbol Comparator:LM311
- added U5: 5V Converter, footprint:DCDC_MODULE, symbol A-FA_PARTS:DC-DC_Converter
- added U6: 3.3V Converter, footprint:DCDC_MODULE, symbol A-FA_PARTS:DC-DC_Converter
- added U7: CAN_TRANSCEIVER, footprint:CAN_TRANSIVER, symbol A-FA_PARTS:CAN_TRANSCEIVER
- added U8: D302, footprint:SPK_D302, symbol A-FA_PARTS:D302
- added U9: ADXL345, footprint:ADXL345, symbol A-FA_PARTS:ADXL345
Connections:
- net 3.3V: now also R33.2, R34.2, R35.2, R36.2, R52.2, R53.2, R54.2, R55.2, R56.2, SW9.1, U10.1 (VCC), U11.2 (3V3), U6.3 (OUT), U7.1 (3V3), U9.1 (3V3), U9.7 (~{CS})
- net ADC2_IN0: now also J10.2 (Pin_2), U15.23 (PA0)
- net ADC2_IN1: now also J10.7 (Pin_7), U15.24 (PA1)
- net ADC2_IN2: now also J9.2 (Pin_2), U15.25 (PA2)
- net ADC2_IN3: now also J9.7 (Pin_7), U15.26 (PA3)
- net ADC3_IN10: now also J10.5 (Pin_5), R5.1, U15.15 (PC0)
- net ADC3_IN11: now also J10.10 (Pin_10), R6.1, U15.16 (PC1)
- net ADC3_IN12: now also J9.5 (Pin_5), R7.1, U15.17 (PC2)
- net ADC3_IN13: now also J9.10 (Pin_10), R8.1, U15.18 (PC3)
- net AIR+: now also J2.3 (Pin_3), K3.14, K4.2, K4.7, K4.8
- net AIR-: now also D10.2 (A), J1.10 (Pin_10), J2.4 (Pin_4), J8.1 (Pin_1), K2.14, K3.7, K3.8, R24.1
- net AIR_DRIVE: now also J1.12 (Pin_12), K3.2
- net BMS_FAULT: now also J2.5 (Pin_5), Q2.1 (G), R9.1
- net BMS_Pin: now also Q8.3 (C), R34.1, U15.59 (PD12)
- net BOTS_{1}: now also J3.2 (Pin_2), J4.3 (Pin_3), J8.10 (Pin_10), J8.15 (Pin_15)
- net BOTS_{2}: now also C1.1, C2.1, J10.4 (Pin_4), J10.9 (Pin_9), J2.1 (Pin_1), J4.4 (Pin_4), J6.1 (Pin_1), J8.4 (Pin_4), J9.4 (Pin_4), J9.9 (Pin_9), K1.7, K1.8, Q5.3 (C), R1.1, R20.1, R21.2, R30.2, R31.2, RLY1.3 (A3), RLY1.4 (11), RLY2.3 (A3), RLY2.4 (11), RLY3.3 (A3), RLY3.4 (11), U2.8 (V+), U3.8 (V+), U5.1 (IN), U6.1 (IN)
- net BRAKE_LIGHT-: now also J1.2 (Pin_2), J8.11 (Pin_11), Q1.2 (D)
- net BSPD_Pin: now also Q10.3 (C), R36.1, U15.61 (PD14)
- net CAN1_{TX}: now also U15.82 (PD1), U7.3 (CTX)
- net CAN_H_{BMS}: now also J2.11 (Pin_11), SW3.6
- net CAN_H_{INV}: now also J1.5 (Pin_5), SW4.6
- net CAN_H_{LOGGER}: now also J3.7 (Pin_7), SW5.6
- net CAN_L_{BMS}: now also J2.12 (Pin_12), SW3.3
- net CAN_L_{INV}: now also J1.6 (Pin_6), SW4.3
- net CAN_L_{LOGGER}: now also J3.8 (Pin_8), SW5.3
- net ESP_RX: now also J11.2 (Pin_2), U11.34 (RXD0)
- net ESP_TX: now also J11.1 (Pin_1), U11.35 (TXD0)
- net FORWARD_ENABLE: now also J1.1 (Pin_1), K6.8
- net GND: now also C6.2, D1.1 (K), D11.1 (K), D12.1 (K), D13.1 (K), D14.1 (K), D15.1 (K), D16.1 (K), D17.1 (K), D2.1 (K), D3.1 (K), D4.1 (K), D5.1 (K), D6.1 (K), D8.1 (K), D9.1 (K), J1.11 (Pin_11), J1.3 (Pin_3), J1.9 (Pin_9), J10.3 (Pin_3), J10.8 (Pin_8), J11.6 (Pin_6), J2.2 (Pin_2), J3.5 (Pin_5), J4.2 (Pin_2), J5.4 (Pin_4), J7.3 (Pin_3), J7.6 (Pin_6), J8.14 (Pin_14), J8.2 (Pin_2), J9.3 (Pin_3), J9.8 (Pin_8), K1.6, K2.6, K3.6, K6.15, K6.16, K6.4, Q1.3 (S), Q10.1 (E), Q12.3 (E), Q13.3 (E), Q14.1 (E), Q4.3 (S), Q7.1 (E), Q8.1 (E), Q9.1 (E), R17.1, R18.2, R22.2, R23.2, R25.2, R3.1, R44.1, R5.2, R6.2, R7.2, R8.2, RV1.2, RV2.2, SW2.1, SW8.2, U1.1 (GND), U10.4 (GND), U11.1 (GND), U11.15 (GND), U11.38 (GND), U11.39_1 (GND), U11.39_10 (GND), U11.39_11 (GND), U11.39_12 (GND), U11.39_13 (GND), U11.39_14 (GND), U11.39_15 (GND), U11.39_16 (GND), U11.39_17 (GND), U11.39_18 (GND), U11.39_19 (GND), U11.39_2 (GND), U11.39_20 (GND), U11.39_21 (GND), U11.39_3 (GND), U11.39_4 (GND), U11.39_5 (GND), U11.39_6 (GND), U11.39_7 (GND), U11.39_8 (GND), U11.39_9 (GND), U12.10 (GND_2), U12.7 (GND_1), U13.1 (GND), U14.1 (GND), U2.1 (GND), U2.4 (V-), U3.1 (GND), U3.4 (V-), U5.2 (GND), U5.4 (GND), U6.2 (GND), U6.4 (GND), U7.2 (GND), U8.2 (GND), U8.8 (GND), U9.2 (GND)
- net GPS_{RX}: now also U10.2 (RX), U15.63 (PC6)
- net HV_ACTIVE_Pin: now also Q7.3 (C), R33.1, U15.58 (PD11)
- net HV_AUX_{L2}: now also J4.6 (Pin_6), R4.1, RLY1.7 (21)
- net HV_MASTER_{1}: now also J3.3 (Pin_3), RLY3.8 (22)
- net HV_MASTER_{2}: now also J3.4 (Pin_4), K2.7, K2.8
- net IMD_FAULT: now also J2.6 (Pin_6), Q3.1 (G), R12.2
- net IMD_Pin: now also Q9.3 (C), R35.1, U15.60 (PD13)
- net LV+: now also F1.2, J4.1 (Pin_1)
- net LV_MASTER_{1}: now also F1.1, J3.1 (Pin_1)
- net RTD_ACTIVE_Pin: now also Q14.3 (C), R55.1, U15.57 (PD10)
- net RTD_BUTTON: now also J5.7 (Pin_7), K5.6
- net RTD_LED: now also J5.8 (Pin_8), R48.2
- net RTD_RESET: now also K3.1, K6.1
- net SPK_L+: now also J8.6 (Pin_6), U8.3 (LOUT+)
- net SPK_L-: now also J8.7 (Pin_7), U8.4 (LOUT-)
- net SPK_R+: now also J8.8 (Pin_8), U8.6 (ROUT+)
- net SPK_R-: now also J8.9 (Pin_9), U8.5 (ROUT-)
- new net: D5.2 (A), Q3.2 (D)
- new net: C6.1, R46.1, U14.6 (THR), U14.7 (DIS)
- new net: K6.9, R46.2, R47.1, R48.1, R49.1, R50.2, R51.2, U14.4 (R), U14.8 (VCC)
- new net: Q14.2 (B), R47.2
- new net: D2.2 (A), Q2.3 (S)
- new net: SW8.1, U11.25 (IO0)
- new net: 10uF1.1, K1.14, U1.4 (R), U1.8 (VCC)
- new net: 10uF1.2, R18.1, U1.2 (TR), U1.6 (THR)
- new net: Q12.1 (C), U12.11 (IO_2)
- new net: U12.4 (DAC_R), U8.7 (RIN)
- new net: U12.5 (DAC_L), U8.9 (LIN)
- new net: SW3.1, SW4.1, SW5.1, SW6.1, SW7.1
- new net: SW3.4, SW4.4, SW5.4, SW6.4, SW7.4
- new net: C4.1, R23.1, R32.1, U3.2 (+)
- new net: C4.2, R31.1, RV2.1, U3.3 (-)
- new net: Q4.1 (G), R17.2, U1.3 (Q)
- new net: D7.1 (K), Q4.2 (D)
- new net: C3.1, R22.1, R29.1, U2.2 (+)
- new net: C3.2, R30.1, RV1.1, U2.3 (-)
- new net: C5.2, R44.2, U13.2 (TR), U13.6 (THR)
- new net: K6.2, U13.3 (Q)
- new net: C5.1, K5.14, K6.13, U13.4 (R), U13.8 (VCC)
- new net: C1.2, U2.5 (BAL), U2.6 (STRB)
- new net: Q13.1 (C), R50.1, U14.2 (TR)
- new net: R45.2, U14.3 (Q)
- new net: Q10.2 (B), R26.2
- new net: Q5.1 (E), Q6.3 (C)
- new net: Q5.2 (B), R20.2, U2.7
- new net: D7.2 (A), RLY3.2 (A2)
- new net: D14.2 (A), R41.2
- new net: C2.2, U3.5 (BAL), U3.6 (STRB)
- new net: Q6.2 (B), R21.1, U3.7
- new net: SW9.2, U15.94 (BOOT0)
- new net: Q3.3 (S), R12.1, RLY2.2 (A2)
- new net: R13.1, RLY2.5 (12)
- new net: R14.1, R27.1, RLY2.6 (14)
- new net: RLY1.8 (22), RLY2.7 (21)
- new net: RLY2.8 (22), RLY3.7 (21)
- new net: R15.1, RLY3.5 (12)
- new net: D8.2 (A), R15.2
- new net: R16.1, R26.1, RLY3.6 (14)
- new net: Q7.2 (B), R24.2
- new net: D3.2 (A), R4.2
- new net: K4.14, K5.7, K5.8, Q11.1 (C), U8.1 (VIN)
- new net: AE1.1 (A), U10. (A)
- new net: J1.7 (Pin_7), J7.4 (Pin_4)
- new net: J1.8 (Pin_8), J7.5 (Pin_5)
- new net: J2.10 (Pin_10), J5.12 (Pin_12)
- new net: J2.7 (Pin_7), J5.9 (Pin_9)
- new net: J2.8 (Pin_8), J5.10 (Pin_10)
- new net: J2.9 (Pin_9), J5.11 (Pin_11)
- new net: K1.2, Q6.1 (E), R19.1
- new net: SW7.3, U7.6 (CANL)
- new net: SW7.6, U7.5 (CANH)
- new net: D11.2 (A), R38.2
- new net: R11.1, R28.1, RLY1.6 (14)
- new net: Q8.2 (B), R28.2
- new net: Q1.1 (G), R2.1
- new net: D6.2 (A), R13.2
- new net: R40.1, U15.43 (PE12)
- new net: D13.2 (A), R40.2
- new net: Q9.2 (B), R27.2
- new net: D4.2 (A), R10.2
- new net: Q12.2 (B), R45.1
- new net: Q11.2 (B), R37.2
- new net: J1.4 (Pin_4), J12.1 (Pin_1)
- new net: D10.1 (K), R25.1
- new net: Q2.2 (D), R9.2, RLY1.2 (A2)
- new net: R10.1, RLY1.5 (12)
- new net: Q13.2 (B), R51.1
- new net: D9.2 (A), R19.2
- new net: R42.1, U15.45 (PE14)
- new net: D15.2 (A), R42.2
- new net: SW2.2, U11.3 (EN)
- new net: D17.2 (A), R49.2
- new net: R39.1, U15.42 (PE11)
- new net: D12.2 (A), R39.2
- new net: R38.1, U15.41 (PE10)
- new net: R41.1, U15.44 (PE13)
- new net: R43.1, U15.46 (PE15)
- new net: D16.2 (A), R43.2
- new net: K5.2, Q11.3 (E)
- new net: D1.2 (A), R1.2
- new net ACC_{SCL}: R53.1, U15.67 (PA8), U9.14 (SCL/SCLK)
- new net ACC_{SDA}: R56.1, U15.66 (PC9), U9.13 (SDA)
- new net BRAKE_SW_{2}: J8.16 (Pin_16), R2.2, R3.2, R37.1
- new net BRAKE_{PWR}: J10.1 (Pin_1), J10.6 (Pin_6), J5.14 (Pin_14), J8.12 (Pin_12), J9.1 (Pin_1), J9.6 (Pin_6), R57.2, R58.2, U12.1 (VCC), U15.100 (VDD), U5.3 (OUT)
- new net BRAKE_{SIG}: J8.13 (Pin_13), R29.2
- new net CAN1_{RX}: U15.81 (PD0), U7.4 (CRX)
- new net CAN_H_{DEBUG}: J7.1 (Pin_1), SW6.6
- new net CAN_L_{DEBUG}: J7.2 (Pin_2), SW6.3
- new net ESP_{SCL}: R54.1, U11.36 (IO22), U15.93 (PB7)
- new net ESP_{SDA}: R52.1, U11.33 (IO21), U15.92 (PB6)
- new net GPS_{TX}: U10.3 (TX), U15.64 (PC7)
- new net HALL_{SIG}: J8.3 (Pin_3), R32.2
- new net HVD_{2}: J8.5 (Pin_5), K2.2
- new net HV_AUX_{L1}: J4.5 (Pin_5), J4.8 (Pin_8)
- new net HV_AUX_{R1}: J4.7 (Pin_7), J6.2 (Pin_2)
- new net LATCH_{BMS}: J5.3 (Pin_3), R11.2
- new net LATCH_{BSPD}: J5.1 (Pin_1), R16.2
- new net LATCH_{IMD}: J5.2 (Pin_2), R14.2
- new net LCD_{SCL}: J5.16 (Pin_16), R57.1, U15.47 (PB10)
- new net LCD_{SDA}: J5.15 (Pin_15), R58.1, U15.48 (PB11)
- new net RESET_{2}: J3.6 (Pin_6), RLY1.1 (A1), RLY2.1 (A1), RLY3.1 (A1)
- new net STM_{RX}: J11.5 (Pin_5), U15.69 (PA10)
- new net STM_{TX}: J11.4 (Pin_4), U15.68 (PA9)
- new net SW_{RTD_EN}: J5.13 (Pin_13), K4.6
- no-connect marks 129 -> 128
Other:
- note removed: "EXTERNAL INTERFACE PIN"
- note removed: "INTERFACES"
- note removed: "INTERNAL CIRCUIT PIN"
- note removed: "INTERNAL STM32 PIN"
- note removed: "PIN SHAPE DEFINITION"

Commit message: update: schematics and wirings to current state
Other:
- note added: "Actual Measurement ON 0V OFF 3.3V"
- note added: "Actual Measurement ON 3.3V OFF 0.8V"
- note added: "Actual Measurement ON 3.3V OFF 1V"
- note added: "Actual Measurement ON 3V OFF 0.5V"
- note added: "ON GND OFF 2.9V"
- note added: "ON_{BATT_FAN"
- note added: "ON_{COOLING"
- note added: "ON_{PUMP"
- note added: "ON_{RAD_FAN"
- note added: "RS232_{RX"
- note added: "RS232_{TX"
- moved on the sheet: J1, J10, J11, J12, J2, J3, J4, J5, J7, J8, J9
