File: PCBs/LV_PCB v2/LV_PCB.kicad_sch (KiCad schematic)
At the start: 159 parts, among them J1 5267-12AX, J10 5267-12AX, J11 Conn_01x02_Female, J12 5267-12AX, J13 Conn_01x02_Female, J2 5267-12AX, J3 5267-08AX, J4 5267-12AX, J5 Conn_01x14_Female, J6 Conn_01x04_Female, J7 5267-10AX, J8 Conn_01x02_Female, J9 RTDS_{TIM, K1 HR702NH-DC12V, K2 HR702NH-DC12V, K3 HR702NH-DC12V, K4 HR702NH-DC12V, K5 HR702NH-DC12V, K6 HR90L2_12V, Q1 IRF640, Q10 2N3904, Q11 2N3904, Q12 2N3904, Q13 2N3904, Q14 2N3904, Q2 IRF640, Q3 IRF9540N, Q4 IRF640, Q5 2N3904, Q6 2N3904, Q7 IRF640, Q8 2N3904, Q9 2N3904, SW1 CAN_{DEBUG, SW2 CAN_{ECU, SW3 CAN_{BMS, SW4 CAN_{INV, SW5 CAN_{LOGGER, SW8 ESP_{PROGRAM, U1 NE555D, U10 NEO-7M, U11 ESP32-WROOM-32D, U12 DFR0299, U13 LM555xN, U14 LM555xN, U15 STM32F407VETx, U16 LM311, U17 LM311, U18 LM311, U19 LM311, U2 LM311, U3 LM311, U4 AMS1117-3.3, U5 5V Converter, U6 3.3V Converter, U7 CAN_TRANSCEIVER, U8 D302, U9 ADXL345

Commit message: update: 23/08/14
Parts:
- removed D1: OK_{LV, LED_THT:LED_D5.0mm, symbol Device:LED
- removed R1: 5k, Resistor_THT:R_Axial_DIN0207_L6.3mm_D2.5mm_P10.16mm_Horizontal, symbol Device:R_US
- added C?: 1000uF, Capacitor_THT:C_Disc_D5.0mm_W2.5mm_P2.50mm, symbol Device:C_Small
- added D?: OK_{LV, LED_THT:LED_D5.0mm, symbol Device:LED
- added R?: 4.7k, Resistor_THT:R_Axial_DIN0207_L6.3mm_D2.5mm_P10.16mm_Horizontal, symbol Device:R_US
- R2: value 100k -> 1k
- R24, R5: value 5k -> 4.7k
Connections:
- net BOTS_{2}: now also R?.1
- net CAN_H_{INV}: now also SW4.6; no longer SW4.3
- net CAN_L_{INV}: now also SW4.3; no longer SW4.6
- net GND: now also C?.2, D?.1 (K)
- net LV+: now also C?.1
- net RTD_RESET: now reaches K2.1, K6.1
- net IGNITION_INPUT renamed IGNITION
- new net: D?.2 (A), R?.2
Other:
- note added: "When the HV_ACTIVE is engaged, inverter and AIR- is turned on and drains current. This leads significant voltage drop on the LV_{PCB} rail for ~5ms. Following 5V and 3.3V rail's voltage drop causes brownout situation for STM32 and ESP32. This 1000uF cap compensates the drop and make power line stabler."
- note added: "connect one of these jumper to choose the RTDS trigger"
- moved on the sheet: LV-_{CONN
