File: EV.kicad_sch (KiCad schematic)
At the start: 36 parts, among them J1 RS232_SERIAL, J2 RS232_CAN, M1 PUMP, M2 FAN_L, M3 FAN_R, M4 Emrax_208, SW1 PUSH_ROTATE, SW2 RESET_BUTTON, SW3 BRAKE, SW4 BOTS, SW5 HV_AUX_L, SW6 HV_AUX_R, U1 PM100DX_GEN3, U2 LV_Converter

Commit message: update schematics snapshot
Connections:
- net at M4. (TH): now also U1. (HV-)
- new net: M4. (TH), U1. (HV-) (x2)
Other:
- sheet CHARGE SHUTDOWN: file CHARGE SHUTDOWN.kicad_sch -> PCBs/CHARGE_SHUTDOWN/CHARGE_SHUTDOWN.kicad_sch
- sheet JUNCTION: file JUNCTION.kicad_sch -> PCBs/JUNCTION/JUNCTION.kicad_sch

Commit message: update: schematics and wirings to current state
Connections:
- net at M4. (TH): now also U1. (HV-)
- new net: M4. (TH), U1. (HV-) (x2)
Changed lines of the file:
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@@
     )
     (path "/955faa4e-8420-4c3f-8749-c4fc7f2d01e7/e0d16234-8d73-45f3-ae88-98a3a2553b31/f5d5bc02-07f8-4ce6-84d4-81dc26ac83f7"
-      (reference "F2") (unit 1) (value "1A Fuse") (footprint "Fuse:Fuseholder_Cylinder-5x20mm_Schurter_0031_8201_Horizontal_Open")
+      (reference "F2") (unit 1) (value "3A Fuse") (footprint "Fuse:Fuseholder_Cylinder-5x20mm_Schurter_0031_8201_Horizontal_Open")
     )
     (path "/955faa4e-8420-4c3f-8749-c4fc7f2d01e7/e0d16234-8d73-45f3-ae88-98a3a2553b31/98b83cf6-cd62-486b-8e4f-fb0b58e00050"
-      (reference "F3") (unit 1) (value "3A Fuse") (footprint "Fuse:Fuseholder_Cylinder-5x20mm_Schurter_0031_8201_Horizontal_Open")
+      (reference "F3") (unit 1) (value "1A Fuse") (footprint "Fuse:Fuseholder_Cylinder-5x20mm_Schurter_0031_8201_Horizontal_Open")
     )
     (path "/955faa4e-8420-4c3f-8749-c4fc7f2d01e7/e0d16234-8d73-45f3-ae88-98a3a2553b31/19474afc-0870-4fc1-9fed-29743a44d1d1"
@@
       (reference "J6") (unit 1) (value "Conn_01x02_Female") (footprint "footprint:5566-02A")
     )
+    (path "/a801bf24-47be-44f6-9278-ef6290da97dd/683f4176-7a4b-4891-9155-0d79666ebacb"
+      (reference "J6") (unit 1) (value "ENERGYMETER") (footprint "Connector_PinHeader_2.54mm:PinHeader_1x02_P2.54mm_Vertical")
+    )
     (path "/955faa4e-8420-4c3f-8749-c4fc7f2d01e7/a63d25dc-917a-4b49-a75d-911b11a1500c"
       (reference "J6") (unit 1) (value "Conn_01x01_Male") (footprint "")
@@
       (reference "J7") (unit 1) (value "5267-06AX") (footprint "Connector_PinHeader_2.54mm:PinHeader_1x06_P2.54mm_Vertical")
     )
+    (path "/a801bf24-47be-44f6-9278-ef6290da97dd/9cf25dfd-c37b-4cad-b8ee-d1e84098b796"
+      (reference "J7") (unit 1) (value "R_DISCHARGE") (footprint "Connector_PinHeader_2.54mm:PinHeader_1x01_P2.54mm_Vertical")
+    )
     (path "/955faa4e-8420-4c3f-8749-c4fc7f2d01e7/a99bc7dd-4774-4b2f-beb8-7f6f2ea5e60c"

Commit message: fix: broken LV_PCB link
Connections:
- net at M4. (TH): now also U1. (HV-)
- new net: M4. (TH), U1. (HV-) (x2)
Other:
- sheet LV PCB: file PCBs/LV_PCB/LV_PCB.kicad_sch -> PCBs/LV_PCB v2/LV_PCB.kicad_sch
