File: HV_BATT.kicad_sch (KiCad schematic)
At the start: 38 parts, among them J10 Conn_01x01_Female, J11 Conn_01x01_Female, J12 Conn_01x01_Male, J13 Conn_01x03_Female, J14 Conn_01x03_Male, J15 Conn_01x03_Female, J16 Conn_01x03_Male, J17 Conn_01x02_Female, J18 Conn_01x02_Male, J19 Conn_01x02_Male, J20 Conn_01x02_Female, J21 Conn_01x02_Female, J22 Conn_01x02_Male, J23 Conn_01x06_Male, J24 Conn_01x08_Male, J25 Conn_01x08_Female, J26 Conn_01x06_Female, J27 Conn_01x09_Male, J28 Conn_01x09_Female, J29 Conn_01x12_Female, J3 Conn_01x01_Male, J30 Conn_01x12_Male, J4 Conn_01x01_Female, J5 Conn_01x01_Female, J6 Conn_01x01_Male, J7 Conn_01x01_Male, J8 Conn_01x01_Female, J9 Conn_01x01_Male, M5 BATT_FAN, U3 IR155-3204, U4 OrionBMS2-72

Commit message: update schematics snapshot
Connections:
- new net: J13., J14. (x2)
- new net: J15., J16. (x2)

Commit message: update: schematics and wirings to current state
Connections:
- new net: J13., J14. (x2)
- new net: J15., J16. (x2)

Commit message: fix: broken LV_PCB link
Connections:
- new net: J13., J14. (x2)
- new net: J15., J16. (x2)
